File: EDITABLES/PCB/LATEST/PCB_final/DoubLayerSim.sch (KiCad schematic (older format))
At the start: 28 parts, among them J1 PanelSolar, J2 Bateria 3.7v, Q1 2N3904

Commit message: Update 15 JUN
Parts:
- added Q?: Q_PMOS_DGS, symbol Device:Q_PMOS_DGS
- added R? (x4): R, pcb_ss:ResistorPCB, symbol Device:R
Connections:
- net +3V8: no longer SIM1.1 (VCC)
- net GND: now also Q?.3 (S), R?.2; no longer R4.2, SD1.1 (IN-), SIM1.5 (GND)
- net RX: now reaches APM1.7 (D4), R5.1
- net TX: now reaches APM1.8 (D5), SIM1.4 (TXD)
- net at SIM1.6 (DTR): no longer APM1.9 (D6)
- net at SIM1.2 (RST): now also R?.2, R?.2
- new net: Q?.2 (G), R?.1
- new net: R?.1, R?.2
- new net 4.4V_REG: SIM1.1 (VCC)
- new net GND_SIM: Q?.1 (D), R4.2, R?.1, SIM1.5 (GND)
- new net RST: APM1.9 (D6), R?.1
- now unconnected: J1.2 (Pin_2), R3.2, SD1.2 (IN+)
- no-connect marks 8 -> 7
Other:
- moved on the sheet: R3, R4, R5, R6, R8, R9, SD1, SIM1, SU1, TP1
